File: Circuit/TechnoVikingPCB.kicad_sch (KiCad schematic)
At the start: 122 parts, among them Q1 SQ4005EY-T1_BE3, Q2 BSS315PH6327XTSA1, Q3 BSS315PH6327XTSA1, Q4 BSS315PH6327XTSA1, U1 LMV324, U2 LMV324, X1 Conn_01x02_Male, X2 Conn_01x05_Male, X3 Conn_01x02_Male, X4 Conn_01x02_Male, X5 Conn_01x02_Female, X6 Conn_01x02_Male, X7 Conn_01x04_Male, X8 Conn_01x03_Male, X9 Conn_01x03_Male

Commit message: Documentation.
Parts:
- D4, D5, D9: value NSR0320MW2T1G -> PMEG4010BEA,115
- MK1: value Microphone_Condenser -> CMEJ-0627-42-P
- Q2, Q3, Q4: value BSS315PH6327XTSA1 -> BSH105,215
Other:
- note removed: "Relpaced"
Changed lines of the file:
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@@
     (effects (font (size 2.54 2.54) (thickness 0.254) bold) (justify left bottom))
   )
-  (text "Relpaced\n" (at 347.98 214.63 0)
-    (effects (font (size 1.27 1.27)) (justify left bottom))
-  )
   (text "Endstops\n" (at 243.205 76.835 0)
     (effects (font (size 3.81 3.81) (thickness 0.254) bold) (justify left bottom))
   )
-  (text "Relpaced\n" (at 363.855 119.38 0)
-    (effects (font (size 1.27 1.27)) (justify left bottom))
-  )
   (text "LED-strip interface\n" (at 243.205 197.485 0)
     (effects (font (size 3.81 3.81) (thickness 0.254) bold) (justify left bottom))
@@
     (effects (font (size 3.81 3.81) (thickness 0.254) bold) (justify left bottom))
   )
-  (text "Relpaced\n" (at 354.965 237.49 0)
-    (effects (font (size 1.27 1.27)) (justify left bottom))
-  )
   (text "Buzzer driver\n" (at 360.68 76.2 0)
     (effects (font (size 3.81 3.81) (thickness 0.254) bold) (justify left bottom))
@@
     (effects (font (size 1.524 1.524) italic) (justify left bottom))
   )
-  (text "Relpaced\n" (at 354.33 100.33 0)
-    (effects (font (size 1.27 1.27)) (justify left bottom))
-  )
   (text "Analog stage" (at 20.955 175.895 0)
     (effects (font (size 5.08 5.08) (thickness 0.254) bold) (justify left bottom))
@@
     (effects (font (size 3.81 3.81) (thickness 0.254) bold) (justify left bottom))
   )
-  (text "Relpaced\n" (at 348.615 156.21 0)
-    (effects (font (size 1.27 1.27)) (justify left bottom))
-  )
   (text "Half-wave rectifier\nwith analog buffer\nfor signal level\ndetection"
     (at 146.685 33.02 0)
     (effects (font (size 2.54 2.54) (thickness 0.254) bold) (justify left bottom))
   )
-  (text "Relpaced\n" (at 355.6 179.705 0)
-    (effects (font (size 1.27 1.27)) (justify left bottom))
-  )
   (text "DC-Motor driver\n" (at 351.79 139.7 0)
     (effects (font (size 3.81 3.81) (thickness 0.254) bold) (justify left bottom))
@@
       (effects (font (size 1.27 1.27)) (justify left))
     )
-    (property "Value" "NSR0320MW2T1G" (id 1) (at 365.76 86.995 0)
+    (property "Value" "PMEG4010BEA,115" (id 1) (at 365.76 86.995 0)
       (effects (font (size 1.27 1.27)) (justify left))
     )
@@
       (effects (font (size 1.27 1.27)) hide)
     )
-    (property "Datasheet" "https://www.onsemi.com/pdf/datasheet/nsr0320mw2t1-d.pdf" (id 3) (at 360.045 95.25 0)
+    (property "Datasheet" "https://assets.nexperia.com/documents/data-sheet/PMEG4010BEA.pdf" (id 3) (at 360.045 95.25 0)
       (effects (font (size 1.27 1.27)) hide)
     )
@@
       (effects (font (size 1.27 1.27)) (justify left))
     )
-    (property "Value" "BSS315PH6327XTSA1" (id 1) (at 355.6 232.4099 0)
+    (property "Value" "BSH105,215" (id 1) (at 355.6 232.4099 0)
       (effects (font (size 1.27 1.27)) (justify left))
     )
@@
       (effects (font (size 1.27 1.27) italic) (justify left) hide)
     )
-    (property "Datasheet" "https://www.mouser.com/datasheet/2/196/Infineon-BSS315P-DS-v02_03-en-1225631.pdf" (id 3) (at 349.25 231.14 0)
+    (property "Datasheet" "https://assets.nexperia.com/documents/data-sheet/BSH105.pdf" (id 3) (at 349.25 231.14 0)
       (effects (font (size 1.27 1.27)) (justify left) hide)
     )
@@
       (effects (font (size 1.27 1.27)) (justify left))
     )
-    (property "Value" "NSR0320MW2T1G" (id 1) (at 333.375 220.345 90)
+    (property "Value" "PMEG4010BEA,115" (id 1) (at 332.105 220.345 90)
       (effects (font (size 1.27 1.27)) (justify left))
     )
@@
       (effects (font (size 1.27 1.27)) hide)
     )
-    (property "Datasheet" "https://www.onsemi.com/pdf/datasheet/nsr0320mw2t1-d.pdf" (id 3) (at 351.79 219.075 0)
+    (property "Datasheet" "https://assets.nexperia.com/documents/data-sheet/PMEG4010BEA.pdf" (id 3) (at 351.79 219.075 0)
       (effects (font (size 1.27 1.27)) hide)
     )
@@
       (effects (font (size 1.27 1.27)) (justify left))
     )
-    (property "Value" "NSR0320MW2T1G" (id 1) (at 333.375 162.56 90)
+    (property "Value" "PMEG4010BEA,115" (id 1) (at 332.105 162.56 90)
       (effects (font (size 1.27 1.27)) (justify left))
     )
@@
       (effects (font (size 1.27 1.27)) hide)
     )
-    (property "Datasheet" "https://www.onsemi.com/pdf/datasheet/nsr0320mw2t1-d.pdf" (id 3) (at 351.79 161.925 0)
+    (property "Datasheet" "https://assets.nexperia.com/documents/data-sheet/PMEG4010BEA.pdf" (id 3) (at 351.79 161.925 0)
       (effects (font (size 1.27 1.27)) hide)
     )
@@
       (effects (font (size 1.27 1.27)) (justify left))
     )
-    (property "Value" "BSS315PH6327XTSA1" (id 1) (at 363.855 115.5699 0)
+    (property "Value" "BSH105,215" (id 1) (at 363.855 115.5699 0)
       (effects (font (size 1.27 1.27)) (justify left))
     )
@@
       (effects (font (size 1.27 1.27) italic) (justify left) hide)
     )
-    (property "Datasheet" "https://www.mouser.com/datasheet/2/196/Infineon-BSS315P-DS-v02_03-en-1225631.pdf" (id 3) (at 357.505 114.3 0)
+    (property "Datasheet" "https://assets.nexperia.com/documents/data-sheet/BSH105.pdf" (id 3) (at 357.505 114.3 0)
       (effects (font (size 1.27 1.27)) (justify left) hide)
     )
@@
       (effects (font (size 1.27 1.27)) (justify left))
     )
-    (property "Value" "Microphone_Condenser" (id 1) (at 28.575 48.1964 0)
+    (property "Value" "CMEJ-0627-42-P" (id 1) (at 28.575 48.1964 0)
       (effects (font (size 1.27 1.27)) (justify left))
     )
@@
       (effects (font (size 1.27 1.27)) (justify left))
     )
-    (property "Value" "BSS315PH6327XTSA1" (id 1) (at 355.6 175.2599 0)
+    (property "Value" "BSH105,215" (id 1) (at 355.6 175.2599 0)
       (effects (font (size 1.27 1.27)) (justify left))
     )
@@
       (effects (font (size 1.27 1.27) italic) (justify left) hide)
     )
-    (property "Datasheet" "https://www.mouser.com/datasheet/2/196/Infineon-BSS315P-DS-v02_03-en-1225631.pdf" (id 3) (at 349.25 173.99 0)
+    (property "Datasheet" "https://assets.nexperia.com/documents/data-sheet/BSH105.pdf" (id 3) (at 349.25 173.99 0)
       (effects (font (size 1.27 1.27)) (justify left) hide)
     )
@@
     )
     (path "/657c8ae0-52f1-45e9-bbd2-114c0df91597"
-      (reference "D4") (unit 1) (value "NSR0320MW2T1G") (footprint "Diode_SMD:D_SOD-323_HandSoldering")
+      (reference "D4") (unit 1) (value "PMEG4010BEA,115") (footprint "Diode_SMD:D_SOD-323_HandSoldering")
     )
     (path "/530eeef4-fb27-44e7-abe5-3792204c8086"
-      (reference "D5") (unit 1) (value "NSR0320MW2T1G") (footprint "Diode_SMD:D_SOD-323_HandSoldering")
+      (reference "D5") (unit 1) (value "PMEG4010BEA,115") (footprint "Diode_SMD:D_SOD-323_HandSoldering")
     )
     (path "/232f43d3-d005-4425-88aa-77cb4f63e9ab"
@@
     )
     (path "/1efed246-338b-452b-8a44-817284d60917"
-      (reference "D9") (unit 1) (value "NSR0320MW2T1G") (footprint "Diode_SMD:D_SOD-323_HandSoldering")
+      (reference "D9") (unit 1) (value "PMEG4010BEA,115") (footprint "Diode_SMD:D_SOD-323_HandSoldering")
     )
     (path "/dbe0d046-fd06-4f53-b49c-5b54f8b1f80f"
@@
     )
     (path "/dfe58802-4e6b-4809-8436-b1385fe893d2"
-      (reference "MK1") (unit 1) (value "Microphone_Condenser") (footprint "microphone_local:Mic 6mm")
+      (reference "MK1") (unit 1) (value "CMEJ-0627-42-P") (footprint "microphone_local:Mic 6mm")
     )
     (path "/91c00c3f-524c-44f4-ad15-e4ab25f81a66"
@@
     )
     (path "/e5097b91-1d35-4c6a-8b61-0827de50c956"
-      (reference "Q2") (unit 1) (value "BSS315PH6327XTSA1") (footprint "Package_TO_SOT_SMD:SOT-23")
+      (reference "Q2") (unit 1) (value "BSH105,215") (footprint "Package_TO_SOT_SMD:SOT-23")
     )
     (path "/2293550f-7ce4-4ef1-9b1e-a2474eed21f7"
-      (reference "Q3") (unit 1) (value "BSS315PH6327XTSA1") (footprint "Package_TO_SOT_SMD:SOT-23")
+      (reference "Q3") (unit 1) (value "BSH105,215") (footprint "Package_TO_SOT_SMD:SOT-23")
     )
     (path "/843bdd14-a158-4932-988c-2228eba20d10"
-      (reference "Q4") (unit 1) (value "BSS315PH6327XTSA1") (footprint "Package_TO_SOT_SMD:SOT-23")
+      (reference "Q4") (unit 1) (value "BSH105,215") (footprint "Package_TO_SOT_SMD:SOT-23")
     )
     (path "/63159235-029e-4033-b985-6b9106ef264f"

Commit message: MPN Fields are added to interactive BOM
Parts:
- A1: MPN (none) -> 61304011121
- BZ1: MPN (none) -> AT-0927-TT-6-R
- C1, C12, C2, C21, C28, C29, C30, C31, C32, C37: MPN (none) -> GRM21BR61C106KE15K
- C10, C11, C16, C19, C22, C26, C27, C33, C34, C35, C36, C5, C6, C7, C8: MPN (none) -> CC0603JRX7R7BB104
- C13, C14, C15, C17, C18, C20, C24, C25, C3, C4, C9: MPN (none) -> CC0603KRX7R7BB103
- C23: MPN (none) -> CC0603KRX7R7BB101
- D1, D2: MPN (none) -> BAT42W-G3-08
- D3: MPN (none) -> SMBJ5.0CA-QH
- D4, D5, D9: MPN (none) -> PMEG4010BEA,115
- D6, D7: MPN (none) -> APT1608SYC/J3-AMT
- D8: MPN (none) -> APT1608ZGC-AMT
- F1: MPN (none) -> 0685P6000-01
- FB1, FB2, FB3, FB4, FB5, FB6, FB7: MPN (none) -> BLM18PG600SZ1D
- Q1: MPN (none) -> SQ4005EY-T1_BE3
- Q2, Q3, Q4: MPN (none) -> BSH105,215
- R1, R12, R8: MPN (none) -> CRCW06032K20FKEAC
- R10, R13, R14, R18, R20, R42, R43, R9: MPN (none) -> CRCW06034K70JNEC
- R11, R19, R24, R25, R26, R27, R28, R29, R3, R30, R31, R33, R34, R35, R38, R39, R4, R40, R41, R46, R48, R7: MPN (none) -> RCG060310K0FKEA
- R15, R16, R17, R22, R23, R44, R45, R6: MPN (none) -> CRCW0603100RJNEAC
- R2, R21, R32, R36, R37, R47: MPN (none) -> CRCW06031K00JNEC
- R5: MPN (none) -> CRCW0603200KFKEAC
- U1, U2: MPN (none) -> LMV324IDR
- X1, X3, X4, X6: MPN (none) -> S2B-PH-K-S (LF)(SN)
- X2: MPN (none) -> S5B-PH-K-S (LF)(SN)
- X5: MPN (none) -> 39357-0002
- X7: MPN (none) -> S4B-PH-K-S (LF)(SN)
- X8, X9: MPN (none) -> B3B-PH-K-S(LF)(SN)
